Commit message: Included multiple needle options. Rqt Gui plugin sets max and min from urdf description

File: smart_template_description/urdf/smart_template.xacro (robot description, xacro)
@@ -3,10 +3,16 @@
   <xacro:macro name="smart_template" params="needle_type">
     <!-- Define limit values for each needle type -->
-    <xacro:property name="insertion_upper_limit" value="0.14"/>
+    <xacro:property name="insertion_upper_limit" value="0.115"/>
     <xacro:if value="${needle_type == 'default'}">
-      <xacro:property name="insertion_upper_limit" value="0.14"/>
+      <xacro:property name="insertion_upper_limit" value="0.115"/>
     </xacro:if>
     <xacro:if value="${needle_type == 'stylet'}">
-      <xacro:property name="insertion_upper_limit" value="0.12"/>
+      <xacro:property name="insertion_upper_limit" value="0.115"/>
+    </xacro:if>
+    <xacro:if value="${needle_type == 'smartneedle'}">
+      <xacro:property name="insertion_upper_limit" value="0.165"/>
+    </xacro:if>
+    <xacro:if value="${needle_type == 'biopsygun'}">
+      <xacro:property name="insertion_upper_limit" value="0.175"/>
     </xacro:if>
     <!-- Include materials -->
