Commit message: Moved .stl files to genter origin at the needle guide. Adjusted URDF file accordingly

File: smart_template_description/urdf/smart_template.urdf.xacro (robot description, xacro)
@@ -7,4 +7,5 @@
    </xacro:smart_template>
    <joint name="base_joint" type="fixed">
+    <origin xyz="0 0 0" rpy="0 0 0"/>
     <parent link="world"/>
     <child link="base_link" />

File: smart_template_description/urdf/smart_template.xacro (robot description, xacro)
@@ -2,8 +2,10 @@
 <robot xmlns:xacro="http://wiki.ros.org/xacro">
   <xacro:macro name="smart_template">
+    <!-- Include materials -->
     <xacro:include filename="$(find smart_template_description)/urdf/materials.xacro" />
+    <!-- Define Links -->
     <link name="base_link">
       <visual>
-        <origin xyz="0 0 -0.025" rpy="0 0 ${-pi/2}"/>
+        <origin xyz="0 0 0" rpy="0 0 ${-pi/2}"/>
         <geometry>
           <mesh filename="package://smart_template_description/meshes/base_link.stl"/>
@@ -39,4 +41,5 @@
       </visual>
     </link>
+    <!-- Define joints -->
     <joint name="vertical_joint" type="prismatic">
       <origin xyz="0 0 0" rpy="0 0 0"/>

Commit message: Included option of multiple needle

File: smart_template_description/urdf/smart_template.urdf.xacro (robot description, xacro)
@@ -1,10 +1,13 @@
 <?xml version="1.0"?>
 <robot xmlns:xacro="http://wiki.ros.org/xacro" name="$(arg name)">
-   <xacro:include filename="$(find smart_template_description)/urdf/smart_template.xacro"/>
-   <!-- create link fixed to the "world" -->
-   <link name="world" />
-   <xacro:smart_template>
-   </xacro:smart_template>
-   <joint name="base_joint" type="fixed">
+  <!-- Argument for needle_type -->
+  <xacro:arg name="needle_type" default="default"/>
+  <!-- smart_template URDF -->
+  <xacro:include filename="$(find smart_template_description)/urdf/smart_template.xacro"/>
+  <xacro:smart_template needle_type="$(arg needle_type)">
+  </xacro:smart_template>
+  <!-- create link fixed to the "world" -->
+  <link name="world" />
+  <joint name="base_joint" type="fixed">
     <origin xyz="0 0 0" rpy="0 0 0"/>
     <parent link="world"/>

File: smart_template_description/urdf/smart_template.xacro (robot description, xacro)
@@ -1,5 +1,13 @@
 <?xml version="1.0"?>
 <robot xmlns:xacro="http://wiki.ros.org/xacro">
-  <xacro:macro name="smart_template">
+  <xacro:macro name="smart_template" params="needle_type">
+    <!-- Define limit values for each needle type -->
+    <xacro:property name="insertion_upper_limit" value="0.14"/>
+    <xacro:if value="${needle_type == 'default'}">
+      <xacro:property name="insertion_upper_limit" value="0.14"/>
+    </xacro:if>
+    <xacro:if value="${needle_type == 'stylet'}">
+      <xacro:property name="insertion_upper_limit" value="0.12"/>
+    </xacro:if>
     <!-- Include materials -->
     <xacro:include filename="$(find smart_template_description)/urdf/materials.xacro" />
@@ -36,5 +44,5 @@
         <origin xyz="0 0 0" rpy="0 0 ${-pi/2}"/>
         <geometry>
-          <mesh filename="package://smart_template_description/meshes/needle_link.stl"/>
+          <mesh filename="package://smart_template_description/meshes/needle_link_${needle_type}.stl"/>
         </geometry>
         <material name="silver"/>
@@ -61,5 +69,5 @@
       <child link="needle_link"/>
       <axis xyz="0.0 1.0 0.0"/>
-      <limit upper="0.1" lower="0.0" effort="100" velocity="100"/>
+      <limit upper="${insertion_upper_limit}" lower="0.0" effort="100" velocity="100"/>
     </joint>
   </xacro:macro>

Commit message: Uncommented world link. Included dummy stl file for world link to avoid error message when loading robot in SlicerROS2

File: smart_template_description/urdf/smart_template.urdf.xacro (robot description, xacro)
@@ -7,6 +7,13 @@
   <xacro:smart_template needle_type="$(arg needle_type)">
   </xacro:smart_template>
-  <!-- create link fixed to the "world"
-  <link name="world" />
+  <!-- create link fixed to the "world" -->
+  <link name="world">
+    <visual>
+      <origin xyz="0 0 0" rpy="0 0 0"/>
+      <geometry>
+        <mesh filename="package://smart_template_description/meshes/world.stl"/>
+      </geometry>
+    </visual>
+  </link>
   <joint name="base_joint" type="fixed">
     <origin xyz="0 0 0" rpy="0 0 0"/>
@@ -14,4 +21,3 @@
     <child link="base_link" />
   </joint>
-  -->
 </robot>

Commit message: Included world_pose listener to update world to base_link accordingly to registration results (via \world_pose TransformStamped msg)

File: smart_template_description/urdf/smart_template.urdf.xacro (robot description, xacro)
@@ -8,12 +8,5 @@
   </xacro:smart_template>
   <!-- create link fixed to the "world" -->
-  <link name="world">
-    <visual>
-      <origin xyz="0 0 0" rpy="0 0 0"/>
-      <geometry>
-        <mesh filename="package://smart_template_description/meshes/world.stl"/>
-      </geometry>
-    </visual>
-  </link>
+  <link name="world" />
   <joint name="base_joint" type="fixed">
     <origin xyz="0 0 0" rpy="0 0 0"/>

Commit message: Included calibration mode with unlimited joints in robot description

File: smart_template_description/urdf/smart_template.urdf.xacro (robot description, xacro)
@@ -4,7 +4,8 @@
   <xacro:arg name="needle_type" default="default"/>
   <xacro:arg name="zframe_config" default="default"/>
+  <xacro:arg name="robot_mode" default="default"/>
   <!-- smart_template URDF -->
   <xacro:include filename="$(find smart_template_description)/urdf/smart_template.xacro"/>
-  <xacro:smart_template needle_type="$(arg needle_type)">
+  <xacro:smart_template needle_type="$(arg needle_type)" robot_mode="$(arg robot_mode)">
   </xacro:smart_template>
   <!-- zFrame URDF -->

File: smart_template_description/urdf/smart_template.xacro (robot description, xacro)
@@ -1,5 +1,5 @@
 <?xml version="1.0"?>
 <robot xmlns:xacro="http://wiki.ros.org/xacro">
-  <xacro:macro name="smart_template" params="needle_type">
+  <xacro:macro name="smart_template" params="robot_mode needle_type">
     <!-- Define limit values for each needle type -->
     <xacro:property name="insertion_upper_limit" value="0.115"/>
@@ -61,5 +61,11 @@
       <child link="vertical_link"/>
       <axis xyz="0.0 0.0 1.0"/>
-      <limit upper="0.025" lower="-0.025" effort="100" velocity="100"/>
+      <!-- conditional limits -->
+      <xacro:if value="$(eval robot_mode == 'calibration')">
+        <limit upper="1e6" lower="-1e6" effort="100" velocity="1e6"/>
+      </xacro:if>
+      <xacro:unless value="$(eval robot_mode == 'calibration')">
+        <limit upper="0.025" lower="-0.025" effort="100" velocity="100"/>
+      </xacro:unless>
       <!-- custom extension -->
       <channel>C</channel>
@@ -71,5 +77,11 @@
       <child link="horizontal_link"/>
       <axis xyz="1.0 0.0 0.0"/>
-      <limit upper="0.03" lower="-0.03" effort="100" velocity="100"/>
+      <!-- conditional limits -->
+      <xacro:if value="$(eval robot_mode == 'calibration')">
+        <limit upper="1e6" lower="-1e6" effort="100" velocity="1e6"/>
+      </xacro:if>
+      <xacro:unless value="$(eval robot_mode == 'calibration')">
+        <limit upper="0.03" lower="-0.03" effort="100" velocity="100"/>
+      </xacro:unless>
       <!-- custom extension -->
       <channel>A</channel>
@@ -81,5 +93,12 @@
       <child link="needle_link"/>
       <axis xyz="0.0 1.0 0.0"/>
-      <limit upper="${insertion_upper_limit}" lower="0.0" effort="100" velocity="100"/>
+      <!-- conditional limits -->
+      <xacro:if value="$(eval robot_mode == 'calibration')">
+        <limit upper="1e6" lower="-1e6" effort="100" velocity="1e6"/>
+      </xacro:if>
+      <xacro:unless value="$(eval robot_mode == 'calibration')">
+        <limit upper="${insertion_upper_limit}" lower="0.0" effort="100" velocity="100"/>
+      </xacro:unless>
+      <!-- custom extension -->
       <channel>B</channel>
       <mm_to_count>-1574.8031</mm_to_count>
