Commit message: Adjusted ZFrameToRobot using experimental data collected in AMIGO

File: smart_template_description/urdf/zframe.xacro (robot description, xacro)
@@ -4,8 +4,9 @@
   <xacro:macro name="zframe" params="zframe_config">
     <xacro:property name="zframe_orientation" value="-1.0 0.0 0.0 0.0 1.0 0.0 0.0 0.0 -1.0"/> <!-- Rotation matrix (row by row) -->
-    <xacro:property name="zframe_position" value="0.0 0.0980 -0.1283"/> <!-- Position (x, y, z) -->
+    <xacro:property name="zframe_position" value="0.005 0.1012 -0.1130"/> <!-- Position (x, y, z) -->
     <!-- Define zframe_position based on zframe_config -->
     <xacro:if value="${zframe_config == 'default'}">
-      <xacro:property name="zframe_position" value="0.0 0.0980 -0.1283"/> <!-- Position (x, y, z) -->
+      <xacro:property name="zframe_orientation" value="-0.9991865251176608 -0.0227471589597594 0.03329936281010742 -0.021473120893579854 0.9990420341682031 0.03813030515513918 -0.03413481814365832 0.037384247883267614 -0.9987178325638667"/> <!-- Rotation matrix (row by row) -->
+      <xacro:property name="zframe_position" value="0.0012116279772463 0.10551172656992 -0.11125511768768"/> <!-- Position (x, y, z) -->
     </xacro:if>
     <xacro:if value="${zframe_config == 'old'}"> <!-- SmartNeedle Animal Experiment -->
@@ -14,5 +15,5 @@
     <!-- Combine position and orientation into a homogeneous matrix -->
     <xacro:property name="zframe_pose" value="
-      ${zframe_orientation} ${zframe_position.split(' ')[0]}
+      ${zframe_orientation.split(' ')[0]} ${zframe_orientation.split(' ')[1]} ${zframe_orientation.split(' ')[2]} ${zframe_position.split(' ')[0]}
       ${zframe_orientation.split(' ')[3]} ${zframe_orientation.split(' ')[4]} ${zframe_orientation.split(' ')[5]} ${zframe_position.split(' ')[1]}
       ${zframe_orientation.split(' ')[6]} ${zframe_orientation.split(' ')[7]} ${zframe_orientation.split(' ')[8]} ${zframe_position.split(' ')[2]}

Commit message: Adjusted zframe options

File: smart_template_description/urdf/zframe.xacro (robot description, xacro)
@@ -3,15 +3,16 @@
   <!-- ZFrame parameters (zFrame pose with respect to SmartTemplate origin at the needle guide) -->
   <xacro:macro name="zframe" params="zframe_config">
+    <!-- Define zframe if missing zframe_config parameter: based on geometry with 1 LEGO piece at the robot support-->
     <xacro:property name="zframe_orientation" value="-1.0 0.0 0.0 0.0 1.0 0.0 0.0 0.0 -1.0"/> <!-- Rotation matrix (row by row) -->
-    <xacro:property name="zframe_position" value="0.005 0.1012 -0.1130"/> <!-- Position (x, y, z) -->
+    <xacro:property name="zframe_position" value="0.0 0.0980 -0.1283"/> <!-- Position (x, y, z) -->
     <!-- Define zframe_position based on zframe_config -->
-    <xacro:if value="${zframe_config == 'default'}">
+    <xacro:if value="${zframe_config == 'new'}">  <!-- zframe from registration experiment in AMIGO (2025-04-24)-->
       <xacro:property name="zframe_orientation" value="-0.9991865251176608 -0.0227471589597594 0.03329936281010742 -0.021473120893579854 0.9990420341682031 0.03813030515513918 -0.03413481814365832 0.037384247883267614 -0.9987178325638667"/> <!-- Rotation matrix (row by row) -->
       <xacro:property name="zframe_position" value="0.0012116279772463 0.10551172656992 -0.11125511768768"/> <!-- Position (x, y, z) -->
     </xacro:if>
-    <xacro:if value="${zframe_config == 'old'}"> <!-- SmartNeedle Animal Experiment -->
+    <xacro:if value="${zframe_config == 'old'}"> <!-- zframe from SmartNeedle Animal Experiment in 221 Longwood (2023-12-20) -->
       <xacro:property name="zframe_position" value="0.0 0.0590 -0.1190"/> <!-- Position (x, y, z) -->
     </xacro:if>
-    <!-- Combine position and orientation into a homogeneous matrix -->
+    <!-- Combine position and orientation into a homogeneous matrix (just making things easier on 3D Slicer)-->
     <xacro:property name="zframe_pose" value="
       ${zframe_orientation.split(' ')[0]} ${zframe_orientation.split(' ')[1]} ${zframe_orientation.split(' ')[2]} ${zframe_position.split(' ')[0]}

Commit message: Included 4 options for zframe parameter: none(empty), "old", "default" and "new"

File: smart_template_description/urdf/zframe.xacro (robot description, xacro)
@@ -7,10 +7,13 @@
     <xacro:property name="zframe_position" value="0.0 0.0980 -0.1283"/> <!-- Position (x, y, z) -->
     <!-- Define zframe_position based on zframe_config -->
+    <xacro:if value="${zframe_config == 'old'}"> <!-- zframe from SmartNeedle Animal Experiment in 221 Longwood (2023-12-20) -->
+      <xacro:property name="zframe_position" value="0.0 0.0590 -0.1190"/> <!-- Position (x, y, z) -->
+    </xacro:if>
+    <xacro:if value="${zframe_config == 'default'}">  <!-- zframe from registration experiment in AMIGO (2025-04-24)-->
+      <xacro:property name="zframe_position" value="0.005 0.1012 -0.1130"/> <!-- Position (x, y, z) -->
+    </xacro:if>
     <xacro:if value="${zframe_config == 'new'}">  <!-- zframe from registration experiment in AMIGO (2025-04-24)-->
       <xacro:property name="zframe_orientation" value="-0.9991865251176608 -0.0227471589597594 0.03329936281010742 -0.021473120893579854 0.9990420341682031 0.03813030515513918 -0.03413481814365832 0.037384247883267614 -0.9987178325638667"/> <!-- Rotation matrix (row by row) -->
       <xacro:property name="zframe_position" value="0.0012116279772463 0.10551172656992 -0.11125511768768"/> <!-- Position (x, y, z) -->
-    </xacro:if>
-    <xacro:if value="${zframe_config == 'old'}"> <!-- zframe from SmartNeedle Animal Experiment in 221 Longwood (2023-12-20) -->
-      <xacro:property name="zframe_position" value="0.0 0.0590 -0.1190"/> <!-- Position (x, y, z) -->
     </xacro:if>
     <!-- Combine position and orientation into a homogeneous matrix (just making things easier on 3D Slicer)-->

Commit message: Update zFrame options

File: smart_template_description/urdf/zframe.xacro (robot description, xacro)
@@ -3,12 +3,11 @@
   <!-- ZFrame parameters (zFrame pose with respect to SmartTemplate origin at the needle guide) -->
   <xacro:macro name="zframe" params="zframe_config">
-    <!-- Define zframe if missing zframe_config parameter: based on geometry with 1 LEGO piece at the robot support-->
-    <xacro:property name="zframe_orientation" value="-1.0 0.0 0.0 0.0 1.0 0.0 0.0 0.0 -1.0"/> <!-- Rotation matrix (row by row) -->
-    <xacro:property name="zframe_position" value="0.0 0.0980 -0.1283"/> <!-- Position (x, y, z) -->
     <!-- Define zframe_position based on zframe_config -->
-    <xacro:if value="${zframe_config == 'old'}"> <!-- zframe from SmartNeedle Animal Experiment in 221 Longwood (2023-12-20) -->
-      <xacro:property name="zframe_position" value="0.0 0.0590 -0.1190"/> <!-- Position (x, y, z) -->
+    <xacro:if value="${zframe_config == 'default'}">  <!-- zframe based on geometry with 1 LEGO piece at the robot support -->
+      <xacro:property name="zframe_orientation" value="-1.0 0.0 0.0 0.0 1.0 0.0 0.0 0.0 -1.0"/> <!-- Rotation matrix (row by row) -->
+      <xacro:property name="zframe_position" value="0.0 0.0980 -0.1283"/> <!-- Position (x, y, z) -->
     </xacro:if>
-    <xacro:if value="${zframe_config == 'default'}">  <!-- zframe from registration experiment in AMIGO (2025-04-24)-->
+    <xacro:if value="${zframe_config == 'test'}">  <!-- zframe from registration experiment in AMIGO (2025-04-24)-->
+      <xacro:property name="zframe_orientation" value="-1.0 0.0 0.0 0.0 1.0 0.0 0.0 0.0 -1.0"/> <!-- Rotation matrix (row by row) -->
       <xacro:property name="zframe_position" value="0.005 0.1012 -0.1130"/> <!-- Position (x, y, z) -->
     </xacro:if>
@@ -16,4 +15,8 @@
       <xacro:property name="zframe_orientation" value="-0.9991865251176608 -0.0227471589597594 0.03329936281010742 -0.021473120893579854 0.9990420341682031 0.03813030515513918 -0.03413481814365832 0.037384247883267614 -0.9987178325638667"/> <!-- Rotation matrix (row by row) -->
       <xacro:property name="zframe_position" value="0.0012116279772463 0.10551172656992 -0.11125511768768"/> <!-- Position (x, y, z) -->
+    </xacro:if>
+    <xacro:if value="${zframe_config == 'old'}"> <!-- zframe from SmartNeedle Animal Experiment in 221 Longwood (2023-12-20) -->
+      <xacro:property name="zframe_orientation" value="-1.0 0.0 0.0 0.0 1.0 0.0 0.0 0.0 -1.0"/> <!-- Rotation matrix (row by row) -->
+      <xacro:property name="zframe_position" value="0.0 0.0590 -0.1190"/> <!-- Position (x, y, z) -->
     </xacro:if>
     <!-- Combine position and orientation into a homogeneous matrix (just making things easier on 3D Slicer)-->

Commit message: Recalculated zFrame from experiment AMIGO 2025-04-24

File: smart_template_description/urdf/zframe.xacro (robot description, xacro)
@@ -8,11 +8,7 @@
       <xacro:property name="zframe_position" value="0.0 0.0980 -0.1283"/> <!-- Position (x, y, z) -->
     </xacro:if>
-    <xacro:if value="${zframe_config == 'test'}">  <!-- zframe from registration experiment in AMIGO (2025-04-24)-->
-      <xacro:property name="zframe_orientation" value="-1.0 0.0 0.0 0.0 1.0 0.0 0.0 0.0 -1.0"/> <!-- Rotation matrix (row by row) -->
-      <xacro:property name="zframe_position" value="0.005 0.1012 -0.1130"/> <!-- Position (x, y, z) -->
-    </xacro:if>
     <xacro:if value="${zframe_config == 'new'}">  <!-- zframe from registration experiment in AMIGO (2025-04-24)-->
-      <xacro:property name="zframe_orientation" value="-0.9991865251176608 -0.0227471589597594 0.03329936281010742 -0.021473120893579854 0.9990420341682031 0.03813030515513918 -0.03413481814365832 0.037384247883267614 -0.9987178325638667"/> <!-- Rotation matrix (row by row) -->
-      <xacro:property name="zframe_position" value="0.0012116279772463 0.10551172656992 -0.11125511768768"/> <!-- Position (x, y, z) -->
+      <xacro:property name="zframe_orientation" value="-0.9990810696561544 -0.022101423357745315 0.03672187349962075 -0.020810007551375062 0.9991641103988661 0.035185134034339226 -0.037468819763572525 0.03438861763171322 -0.9987059378014156"/> <!-- Rotation matrix (row by row) -->
+      <xacro:property name="zframe_position" value="0.001171932293919652 0.10549880638836385 -0.11120061509823658"/> <!-- Position (x, y, z) -->
     </xacro:if>
     <xacro:if value="${zframe_config == 'old'}"> <!-- zframe from SmartNeedle Animal Experiment in 221 Longwood (2023-12-20) -->

Commit message: New ZFrame transform from 2025-07-23 AMIGO experiment

File: smart_template_description/urdf/zframe.xacro (robot description, xacro)
@@ -8,7 +8,13 @@
       <xacro:property name="zframe_position" value="0.0 0.0980 -0.1283"/> <!-- Position (x, y, z) -->
     </xacro:if>
-    <xacro:if value="${zframe_config == 'new'}">  <!-- zframe from registration experiment in AMIGO (2025-04-24)-->
+    <xacro:if value="${zframe_config == 'test'}">  <!-- zframe from registration experiment in AMIGO (2025-04-24)-->
       <xacro:property name="zframe_orientation" value="-0.9990810696561544 -0.022101423357745315 0.03672187349962075 -0.020810007551375062 0.9991641103988661 0.035185134034339226 -0.037468819763572525 0.03438861763171322 -0.9987059378014156"/> <!-- Rotation matrix (row by row) -->
       <xacro:property name="zframe_position" value="0.001171932293919652 0.10549880638836385 -0.11120061509823658"/> <!-- Position (x, y, z) -->
+    </xacro:if>
+    <xacro:if value="${zframe_config == 'new'}">  <!-- zframe from registration experiment in AMIGO (2025-07-23)-->
+      <xacro:property name="zframe_orientation" value="-0.9996147025670941  0.014578846766073413  0.023618849514765904
+      0.01389168105492629  0.9994828181328841  -0.029001386987696023
+      -0.024029440919981136  -0.028662061839630798  -0.9993002853456078"/> <!-- Rotation matrix (row by row) -->
+      <xacro:property name="zframe_position" value="0.004914398868714972 0.10075025081155526 -0.11873539242196507"/> <!-- Position (x, y, z) -->
     </xacro:if>
     <xacro:if value="${zframe_config == 'old'}"> <!-- zframe from SmartNeedle Animal Experiment in 221 Longwood (2023-12-20) -->

Commit message: Included new registration for ZFrame

File: smart_template_description/urdf/zframe.xacro (robot description, xacro)
@@ -13,7 +13,5 @@
     </xacro:if>
     <xacro:if value="${zframe_config == 'new'}">  <!-- zframe from registration experiment in AMIGO (2025-07-23)-->
-      <xacro:property name="zframe_orientation" value="-0.9996147025670941  0.014578846766073413  0.023618849514765904
-      0.01389168105492629  0.9994828181328841  -0.029001386987696023
-      -0.024029440919981136  -0.028662061839630798  -0.9993002853456078"/> <!-- Rotation matrix (row by row) -->
+      <xacro:property name="zframe_orientation" value="-0.9996147025670941 0.014578846766073413 0.023618849514765904 0.01389168105492629 0.9994828181328841 -0.029001386987696023 -0.024029440919981136 -0.028662061839630798 -0.9993002853456078"/> <!-- Rotation matrix (row by row) -->
       <xacro:property name="zframe_position" value="0.004914398868714972 0.10075025081155526 -0.11873539242196507"/> <!-- Position (x, y, z) -->
     </xacro:if>
